File: pcba/rp2350_gpio_card.kicad_pcb (KiCad board)
At the start: 4 copper layers, 26 x 30 mm, 37 parts, among them J1 Conn_01x10_Pin, J2 Conn_01x10_Pin, P1 USB_C_Plug_USB2.0, U1 RP2350_60QFN, U2 W25Q128JVS, U4 AP2127K-3.3, Y1 ABM8-272-T3

Commit message: 2 layer gerber and minor fix
Parts:
- moved R2 1.05 mm to (99.1, 65.7)
- moved R3 1.05 mm to (99.1, 64.8)
Routing:
- net /USB_D+: track 22.3 -> 25.7 mm
- net /USB_D-: track 21.2 -> 24.4 mm
- net Net-(U1-USB_DM): track 5.50 -> 4.22 mm
- net Net-(U1-USB_DP): track 5.09 -> 4.00 mm
Changed lines of the file:
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@@
 		(tenting front back)
 		(pcbplotparams
-			(layerselection 0x00000000_00000000_55555555_575555f5)
+			(layerselection 0x00000000_00000000_55555555_575555a5)
 			(plot_on_all_layers_selection 0x00000000_00000000_00000000_00000000)
 			(disableapertmacros no)
@@
 			(drillshape 0)
 			(scaleselection 1)
-			(outputdirectory "gerber/")
+			(outputdirectory "gerber2/")
 		)
 	)
@@
 	(footprint "Resistor_SMD:R_0402_1005Metric"
 		(layer "F.Cu")
-		(at 98.05 64.65)
+		(at 99.1 64.75)
 		(descr "Resistor SMD 0402 (1005 Metric), square (rectangular) end terminal, IPC-7351 nominal, (Body size source: IPC-SM-782 page 72, https://www.pcb-3d.com/wordpress/wp-content/uploads/ipc-sm-782a_amendment_1_and_2.pdf), generated with kicad-footprint-generator")
 		(tags "resistor")
@@
 	(footprint "Resistor_SMD:R_0402_1005Metric"
 		(layer "F.Cu")
-		(at 98.05 65.6)
+		(at 99.1 65.7)
 		(descr "Resistor SMD 0402 (1005 Metric), square (rectangular) end terminal, IPC-7351 nominal, (Body size source: IPC-SM-782 page 72, https://www.pcb-3d.com/wordpress/wp-content/uploads/ipc-sm-782a_amendment_1_and_2.pdf), generated with kicad-footprint-generator")
 		(tags "resistor")
@@
 	)
 	(segment
+		(start 99.085 64.15)
+		(end 100.5 64.15)
+		(width 0.127)
+		(layer "F.Cu")
+		(net 1)
+	)
+	(segment
 		(start 100.55 64.2)
 		(end 100.8 64.2)
@@
 	)
 	(segment
-		(start 99.135 64.2)
-		(end 100.55 64.2)
-		(width 0.127)
-		(layer "F.Cu")
-		(net 1)
-	)
-	(segment
 		(start 98.485 63.55)
 		(end 98.5 63.565)
@@
 	)
 	(segment
+		(start 100.5 64.15)
+		(end 100.55 64.2)
+		(width 0.127)
+		(layer "F.Cu")
+		(net 1)
+	)
+	(segment
 		(start 106.7 68.9)
 		(end 108.6 68.9)
@@
 	)
 	(segment
-		(start 109 66.373821)
-		(end 109 65)
-		(width 0.1524)
+		(start 98.5 63.565)
+		(end 99.085 64.15)
+		(width 0.127)
 		(layer "F.Cu")
 		(net 1)
 	)
 	(segment
-		(start 98.5 63.565)
-		(end 99.135 64.2)
-		(width 0.127)
+		(start 109 66.373821)
+		(end 109 65)
+		(width 0.1524)
 		(layer "F.Cu")
 		(net 1)
@@
 	)
 	(segment
-		(start 101.658061 58.3)
-		(end 101.6 58.3)
+		(start 98.54 65.75)
+		(end 98.59 65.7)
 		(width 0.2)
 		(layer "F.Cu")
@@
 	)
 	(segment
-		(start 97.49 65.55)
-		(end 97.54 65.6)
+		(start 101.658061 58.3)
+		(end 101.6 58.3)
 		(width 0.2)
 		(layer "F.Cu")
@@
 	)
 	(segment
-		(start 95.85 65.55)
-		(end 97.49 65.55)
-		(width 0.2)
+		(start 103.305183 54.186434)
+		(end 103.305183 54.971434)
+		(width 0.1524)
 		(layer "F.Cu")
 		(net 28)
 	)
 	(segment
-		(start 103.305183 54.186434)
-		(end 103.305183 54.971434)
-		(width 0.1524)
+		(start 94.75 65.75)
+		(end 98.54 65.75)
+		(width 0.2)
 		(layer "F.Cu")
 		(net 28)
 	)
 	(via
-		(at 95.85 65.55)
+		(at 94.75 65.75)
 		(size 0.6)
 		(drill 0.3)
@@
 	)
 	(segment
-		(start 93.1 61.95)
-		(end 93.1 64.55)
+		(start 92.1 61.7)
+		(end 93.05 60.75)
 		(width 0.2)
 		(layer "B.Cu")
@@
 	)
 	(segment
-		(start 93.1 64.55)
-		(end 94.1 65.55)
+		(start 93.05 60.75)
+		(end 99.15 60.75)
 		(width 0.2)
 		(layer "B.Cu")
@@
 	)
 	(segment
-		(start 94.1 65.55)
-		(end 95.85 65.55)
+		(start 94.75 65.75)
+		(end 93.1 65.75)
 		(width 0.2)
 		(layer "B.Cu")
@@
 	(segment
 		(start 99.15 60.75)
-		(end 94.3 60.75)
+		(end 101.6 58.3)
 		(width 0.2)
 		(layer "B.Cu")
@@
 	)
 	(segment
-		(start 101.6 58.3)
-		(end 99.15 60.75)
+		(start 92.1 64.75)
+		(end 92.1 61.7)
 		(width 0.2)
 		(layer "B.Cu")
@@
 	)
 	(segment
-		(start 94.3 60.75)
-		(end 93.1 61.95)
+		(start 93.1 65.75)
+		(end 92.1 64.75)
 		(width 0.2)
 		(layer "B.Cu")
@@
 	)
 	(segment
-		(start 95.85 64.6)
-		(end 97.49 64.6)
+		(start 98.54 64.8)
+		(end 98.59 64.75)
 		(width 0.2)
 		(layer "F.Cu")
@@
 	)
 	(segment
-		(start 103.805183 57.294817)
-		(end 103.805183 54.961434)
+		(start 94.45 64.8)
+		(end 98.54 64.8)
 		(width 0.2)
 		(layer "F.Cu")
@@
 	)
 	(segment
-		(start 97.49 64.6)
-		(end 97.54 64.65)
+		(start 103.805183 57.294817)
+		(end 103.805183 54.961434)
 		(width 0.2)
 		(layer "F.Cu")
@@
 	)
 	(via
-		(at 103.2 57.9)
-		(size 0.8)
-		(drill 0.4)
+		(at 94.45 64.8)
+		(size 0.6)
+		(drill 0.3)
 		(layers "F.Cu" "B.Cu")
 		(net 29)
 	)
 	(via
-		(at 95.85 64.6)
-		(size 0.6)
-		(drill 0.3)
+		(at 103.2 57.9)
+		(size 0.8)
+		(drill 0.4)
 		(layers "F.Cu" "B.Cu")
 		(net 29)
 	)
 	(segment
-		(start 99.8 61.3)
-		(end 94.65 61.3)
+		(start 94.45 64.8)
+		(end 93.4 64.8)
 		(width 0.2)
 		(layer "B.Cu")
@@
 	)
 	(segment
-		(start 94.25 64.6)
-		(end 95.85 64.6)
+		(start 93.5 61.3)
+		(end 99.8 61.3)
 		(width 0.2)
 		(layer "B.Cu")
@@
 	)
 	(segment
-		(start 93.7 64.05)
-		(end 94.25 64.6)
+		(start 92.75 62.05)
+		(end 93.5 61.3)
 		(width 0.2)
 		(layer "B.Cu")
@@
 	)
 	(segment
-		(start 103.2 57.9)
-		(end 99.8 61.3)
+		(start 93.4 64.8)
+		(end 92.75 64.15)
 		(width 0.2)
 		(layer "B.Cu")
@@
 	)
 	(segment
-		(start 93.7 62.25)
-		(end 93.7 64.05)
+		(start 103.2 57.9)
+		(end 103.2 57.908329)
 		(width 0.2)
 		(layer "B.Cu")
@@
 	)
 	(segment
-		(start 103.2 57.9)
-		(end 103.2 57.908329)
+		(start 92.75 64.15)
+		(end 92.75 62.05)
 		(width 0.2)
 		(layer "B.Cu")
@@
 	)
 	(segment
-		(start 94.65 61.3)
-		(end 93.7 62.25)
+		(start 99.8 61.3)
+		(end 103.2 57.9)
 		(width 0.2)
 		(layer "B.Cu")
@@
 	)
 	(segment
-		(start 102.06623 66.396434)
-		(end 103.317683 66.396434)
-		(width 0.1524)
+		(start 103.317683 66.396434)
+		(end 102.096434 66.396434)
+		(width 0.127)
 		(layer "F.Cu")
 		(net 30)
 	)
 	(segment
-		(start 98.56 65.6)
-		(end 101.269796 65.6)
-		(width 0.1524)
+		(start 101.4 65.7)
+		(end 99.61 65.7)
+		(width 0.127)
 		(layer "F.Cu")
 		(net 30)
 	)
 	(segment
-		(start 101.269796 65.6)
-		(end 102.06623 66.396434)
-		(width 0.1524)
+		(start 102.096434 66.396434)
+		(end 101.4 65.7)
+		(width 0.127)
 		(layer "F.Cu")
 		(net 30)
 	)
 	(segment
-		(start 100.823542 64.7572)
-		(end 98.6672 64.7572)
-		(width 0.1524)
-		(layer "F.Cu")
-		(net 31)
-	)
-	(segment
-		(start 98.691 64.781)
-		(end 98.56 64.65)
-		(width 0.2)
-		(layer "F.Cu")
-		(net 31)
-	)
-	(segment
-		(start 98.6672 64.7572)
-		(end 98.56 64.65)
-		(width 0.1524)
+		(start 103.317683 65.996434)
+		(end 102.121434 65.996434)
+		(width 0.127)
 		(layer "F.Cu")
 		(net 31)
 	)
 	(segment
-		(start 103.317683 65.996434)
-		(end 102.062776 65.996434)
-		(width 0.1524)
+		(start 100.875 64.75)
+		(end 99.61 64.75)
+		(width 0.127)
 		(layer "F.Cu")
 		(net 31)
 	)
 	(segment
-		(start 102.062776 65.996434)
-		(end 100.823542 64.7572)
-		(width 0.1524)
+		(start 102.121434 65.996434)
+		(end 100.875 64.75)
+		(width 0.127)
 		(layer "F.Cu")
 		(net 31)
@@
 	)
 	(segment
-		(start 99.436617 66.5)
-		(end 101.1 66.5)
+		(start 99.609355 66.65)
+		(end 99.615121 66.644234)
 		(width 0.1524)
 		(layer "F.Cu")
@@
 	)
 	(segment
-		(start 98.640183 67.296434)
-		(end 99.436617 66.5)
+		(start 102.596434 67.996434)
+		(end 103.317683 67.996434)
 		(width 0.1524)
 		(layer "F.Cu")
@@
 	)
 	(segment
-		(start 102.596434 67.996434)
-		(end 103.317683 67.996434)
+		(start 101.25 66.65)
+		(end 102.596434 67.996434)
 		(width 0.1524)
 		(layer "F.Cu")
@@
 	)
 	(segment
-		(start 101.1 66.5)
-		(end 102.596434 67.996434)
+		(start 99.286617 66.65)
+		(end 99.609355 66.65)
+		(width 0.1524)
+		(layer "F.Cu")
+		(net 41)
+	)
+	(segment
+		(start 100.211011 66.65)
+		(end 101.25 66.65)
+		(width 0.1524)
+		(layer "F.Cu")
+		(net 41)
+	)
+	(segment
+		(start 100.205245 66.644234)
+		(end 100.211011 66.65)
+		(width 0.1524)
+		(layer "F.Cu")
+		(net 41)
+	)
+	(segment
+		(start 98.640183 67.296434)
+		(end 99.286617 66.65)
+		(width 0.1524)
+		(layer "F.Cu")
+		(net 41)
+	)
+	(segment
+		(start 99.615121 66.644234)
+		(end 100.205245 66.644234)
 		(width 0.1524)
 		(layer "F.Cu")
@@
 	)
 	(segment
-		(start 101.378545 66.2)
+		(start 101.528545 66.35)
 		(end 102.774979 67.596434)
 		(width 0.1524)
@@
 	)
 	(segment
-		(start 97.370183 67.296434)
-		(end 98.466617 66.2)
+		(start 98.316617 66.35)
+		(end 101.528545 66.35)
 		(width 0.1524)
 		(layer "F.Cu")
@@
 	)
 	(segment
-		(start 98.466617 66.2)
-		(end 101.378545 66.2)
+		(start 102.774979 67.596434)
+		(end 103.317683 67.596434)
 		(width 0.1524)
 		(layer "F.Cu")
@@
 	)
 	(segment
-		(start 102.774979 67.596434)
-		(end 103.317683 67.596434)
+		(start 97.370183 67.296434)
+		(end 98.316617 66.35)
 		(width 0.1524)
 		(layer "F.Cu")

Commit message: add no fill zone to L1
Changed lines of the file:
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@@
-	)
-	(segment
-		(start 96.938211 61.92)
-		(end 96.708211 62.15)
-		(width 0.1524)
-		(layer "F.Cu")
-		(net 25)
 	)
 	(segment
@@
 			)
 		)
+	)
+	(zone
+		(net 0)
+		(net_name "")
+		(layer "F.Cu")
+		(hatch edge 0.5)
+		(connect_pads
+			(clearance 0)
+		)
+		(min_thickness 0.25)
+		(filled_areas_thickness no)
+		(keepout
+			(tracks allowed)
+			(vias allowed)
+			(pads allowed)
+			(copperpour not_allowed)
+			(footprints allowed)
+		)
+		(placement
+			(enabled no)
+			(sheetname "")
+		)
+		(fill
+			(thermal_gap 0.5)
+			(thermal_bridge_width 0.5)
+		)
+		(polygon
+			(pts
+				(xy 95.55 61.15) (xy 95.55 64.55) (xy 98.85 64.55) (xy 98.85 61.15)
+			)
+		)
